File: FK9000 Reverse/FK9000 Reverse.kicad_sch (KiCad schematic)
At the start: 4 parts, among them J1 Conn_01x25_Socket

Commit message: Updates
Other:
- note added: "CPU is Toshiba TMP80C50AP 512 Bytes RAM 12 Programmable Functions 14 Bytes per Function 168 Bytes Total Stored in Battery Backed RAM in CPU"
- note added: "Columns: U1_X U1_Y U1_Z U5_X U5_Y Rows: U2_Z U3_X U2_X U2_Y U3_Z U3_Y Pullups on the columns? Only have to scan 5 pins instead of 6?"
- note added: "Crude charge circuit gives about 1-10 mA depending on battery voltage as USB voltage is typically something like ~4.65 volts. Cutoff should be around 4 volts, so should be fine for Li-ion"
- note added: "Line Key R/C U1_Y 0 Key Column U2_Y 0 Key Row U1_Z 1 Key Column U2_Y 1 Key Row U2_Y 2 Key Row U5_Y 2 Key Column U2_Y 3 Key Row U5_X 3 Key Column U1_Z 4 Key Column U2_X 4 Key Row U2_X 5 Key Row U5_Y 5 Key Column U2_X 6 Key Row U5_X 6 Key Column U1_Y 7 Key Column U3_Z 7 Key Row U1_Z 8 Key Column U3_Z 8 Key Row U3_Z 9 Key Row U5_Y 9 Key Column U2_Z AC/On Row U5_X AC/On Column U3_X Asterisk Row U5_X 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"
- note added: "The original boards uses four Toshiba TC4053BP Triple SPDT analog switches. A replacement could be the MC14551B, which would mean only three are needed."
Changed lines of the file:
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@@
+		)
+	)
+	(text "The original boards uses four Toshiba TC4053BP Triple SPDT analog switches.\n\nA replacement could be the MC14551B, which would mean only three are needed.\n\n"
+		(exclude_from_sim no)
+		(at 185.42 142.494 0)
+		(effects
+			(font
+				(size 1.27 1.27)
+			)
+			(justify left)
 		)
 	)
@@
 		(exclude_from_sim no)
 		(at 82.804 43.942 0)
+		(effects
+			(font
+				(size 1.27 1.27)
+			)
+			(justify left)
+		)
+	)
+	(text "Crude charge circuit gives about 1-10 mA depending on battery voltage \nas USB voltage is typically something like ~4.65 volts.\n\nCutoff should be around 4 volts, so should be fine for Li-ion"
+		(exclude_from_sim no)
+		(at 87.376 126.238 0)
 		(effects
 			(font
@@
 		(effects
 			(font
+				(size 1.27 1.27)
+			)
+			(justify left)
+		)
+	)
+	(text "CPU is Toshiba TMP80C50AP\n512 Bytes RAM\n\n12 Programmable Functions\n14 Bytes per Function\n168 Bytes Total\nStored in Battery Backed RAM in CPU"
+		(exclude_from_sim no)
+		(at 165.1 65.024 0)
+		(effects
+			(font
+				(size 1.27 1.27)
+			)
+			(justify left)
+		)
+	)
+	(text "Columns:\nU1_X\nU1_Y\nU1_Z\nU5_X\nU5_Y\n\nRows:\nU2_Z\nU3_X\nU2_X\nU2_Y\nU3_Z\nU3_Y\n\nPullups on the columns?  Only have to scan 5 pins instead of 6?"
+		(exclude_from_sim no)
+		(at 163.322 33.02 0)
+		(effects
+			(font
+				(size 1.27 1.27)
+			)
+			(justify left)
+		)
+	)
+	(text "Line	Key			R/C\nU1_Y	0 Key		Column\nU2_Y	0 Key		Row\nU1_Z	1 Key		Column\nU2_Y	1 Key		Row\nU2_Y	2 Key		Row\nU5_Y	2 Key		Column\nU2_Y	3 Key		Row\nU5_X	3 Key		Column\nU1_Z	4 Key		Column\nU2_X	4 Key		Row\nU2_X	5 Key		Row\nU5_Y	5 Key		Column\nU2_X	6 Key		Row\nU5_X	6 Key		Column\nU1_Y	7 Key		Column\nU3_Z	7 Key		Row\nU1_Z	8 Key		Column\nU3_Z	8 Key		Row\nU3_Z	9 Key		Row\nU5_Y	9 Key		Column\nU2_Z	AC/On		Row\nU5_X	AC/On		Column\nU3_X	Asterisk	Row\nU5_X	Asterisk	Column\nU1_Z	CE			Column\nU2_Z	CE			Row\nU5_X	CE			Column\nU1_X	Delete		Column\nU2_X	Delete		Row\nU2_Y	Divide		Row\nU3_X	Divide		Row\nU5_Y	Divide		Column\nU1_Y	Enter 		Column\nU3_X	Enter 		Row\nU1_Z	M-			Column\nU3_Y	M-			Row\nU1_Z	M+			Column\nU3_X	M+			Row\nU1_X	MC			Column\nU2_Y	MC			Row\nU3_Z	MC			Row\nU3_Z	Minus		Row\nU5_X	Minus		Column\nU1_X	MR			Column\nU3_Y	MR			Row\nU1_Y	Perc		Column\nU3_Y	Perc		Row\nU3_Y	Plus		Row\nU5_X	Plus		Column\nU1_X	Root		Column\nU2_Y	Root		Row"
+		(exclude_from_sim no)
+		(at 240.284 72.136 0)
+		(effects
+			(font
